Commit message: Modified LiDAR height in the xacro; remember to copy it in the description folder of the skidbot and rebuild. Updated package dependencies.

File: xacro/skid.xacro (robot description, xacro)
@@ -153,5 +153,5 @@
         <parent link="chassis"/>
         <child link="laser_frame"/>
-        <origin xyz="0.3 0 0.4" rpy="0 0 0"/> </joint>
+        <origin xyz="0.3 0 0.32" rpy="0 0 0"/> </joint>
     <link name="laser_frame">
         <visual>

Commit message: skid model and train.py for better directories

File: xacro/skid.xacro (robot description, xacro)
@@ -39,5 +39,5 @@
             </geometry>
         </collision>
-        <xacro:inertial_box mass="0.5" x="1.0" y="0.6" z="0.3">
+        <xacro:inertial_box mass="8.0" x="1.0" y="0.6" z="0.3">
             <origin xyz="0 0 0.15" rpy="0 0 0"/>
         </xacro:inertial_box>
@@ -64,6 +64,14 @@
                 <cylinder radius="0.15" length="0.1"/>
             </geometry>
-        </collision>
-        <xacro:inertial_cylinder mass="0.1" length="0.1" radius="0.15">
+            <surface>
+                <friction>
+                    <ode>
+                        <mu>8.0</mu>
+                        <mu2>0.5</mu2>
+                    </ode>
+                </friction>
+            </surface>
+        </collision>
+        <xacro:inertial_cylinder mass="2.0" length="0.1" radius="0.15">
             <origin xyz="0 0 0" rpy="0 0 0"/>
         </xacro:inertial_cylinder>
@@ -90,6 +98,14 @@
                 <cylinder radius="0.15" length="0.1"/>
             </geometry>
-        </collision>
-        <xacro:inertial_cylinder mass="0.1" length="0.1" radius="0.15">
+            <surface>
+                <friction>
+                    <ode>
+                        <mu>8.0</mu>
+                        <mu2>0.5</mu2>
+                    </ode>
+                </friction>
+            </surface>
+        </collision>
+        <xacro:inertial_cylinder mass="2.0" length="0.1" radius="0.15">
             <origin xyz="0 0 0" rpy="0 0 0"/>
         </xacro:inertial_cylinder>
@@ -116,6 +132,14 @@
                 <cylinder radius="0.15" length="0.1"/>
             </geometry>
-        </collision>
-        <xacro:inertial_cylinder mass="0.1" length="0.1" radius="0.15">
+            <surface>
+                <friction>
+                    <ode>
+                        <mu>8.0</mu>
+                        <mu2>0.5</mu2>
+                    </ode>
+                </friction>
+            </surface>
+        </collision>
+        <xacro:inertial_cylinder mass="2.0" length="0.1" radius="0.15">
             <origin xyz="0 0 0" rpy="0 0 0"/>
         </xacro:inertial_cylinder>
@@ -142,6 +166,14 @@
                 <cylinder radius="0.15" length="0.1"/>
             </geometry>
-        </collision>
-        <xacro:inertial_cylinder mass="0.1" length="0.1" radius="0.15">
+            <surface>
+                <friction>
+                    <ode>
+                        <mu>8.0</mu>
+                        <mu2>0.5</mu2>
+                    </ode>
+                </friction>
+            </surface>
+        </collision>
+        <xacro:inertial_cylinder mass="2.0" length="0.1" radius="0.15">
             <origin xyz="0 0 0" rpy="0 0 0"/>
         </xacro:inertial_cylinder>

Commit message: Fixed and added xacro files. Now we have a better dynamic for the skid-steer bot

File: xacro/skid.xacro (robot description, xacro)
@@ -35,9 +35,10 @@
         </visual>
         <collision>
+            <origin xyz="0 0 0.15" rpy="0 0 0"/>
             <geometry>
                 <box size="1.0 0.6 0.3"/>
             </geometry>
         </collision>
-        <xacro:inertial_box mass="8.0" x="1.0" y="0.6" z="0.3">
+        <xacro:inertial_box mass="10.0" x="1.0" y="0.6" z="0.3">
             <origin xyz="0 0 0.15" rpy="0 0 0"/>
         </xacro:inertial_box>
@@ -64,14 +65,6 @@
                 <cylinder radius="0.15" length="0.1"/>
             </geometry>
-            <surface>
-                <friction>
-                    <ode>
-                        <mu>8.0</mu>
-                        <mu2>0.5</mu2>
-                    </ode>
-                </friction>
-            </surface>
-        </collision>
-        <xacro:inertial_cylinder mass="2.0" length="0.1" radius="0.15">
+        </collision>
+        <xacro:inertial_cylinder mass="1.5" length="0.1" radius="0.15">
             <origin xyz="0 0 0" rpy="0 0 0"/>
         </xacro:inertial_cylinder>
@@ -79,6 +72,7 @@
     <gazebo reference="fl_wheel">
         <material>Gazebo/Blue</material>
-        <mu1>20.0</mu1>
-        <mu2>0.1</mu2>
+        <mu1>8.0</mu1>
+        <mu2>0.1</mu2>
+        <fdir1>1 0 0</fdir1>
         <kp>10000000.0</kp>
         <kd>1.0</kd>
@@ -103,14 +97,6 @@
                 <cylinder radius="0.15" length="0.1"/>
             </geometry>
-            <surface>
-                <friction>
-                    <ode>
-                        <mu>8.0</mu>
-                        <mu2>0.5</mu2>
-                    </ode>
-                </friction>
-            </surface>
-        </collision>
-        <xacro:inertial_cylinder mass="2.0" length="0.1" radius="0.15">
+        </collision>
+        <xacro:inertial_cylinder mass="1.5" length="0.1" radius="0.15">
             <origin xyz="0 0 0" rpy="0 0 0"/>
         </xacro:inertial_cylinder>
@@ -118,6 +104,7 @@
     <gazebo reference="fr_wheel">
         <material>Gazebo/Blue</material>
-        <mu1>20.0</mu1>
-        <mu2>0.1</mu2>
+        <mu1>8.0</mu1>
+        <mu2>0.1</mu2>
+        <fdir1>1 0 0</fdir1>
         <kp>10000000.0</kp>
         <kd>1.0</kd>
@@ -142,14 +129,6 @@
                 <cylinder radius="0.15" length="0.1"/>
             </geometry>
-            <surface>
-                <friction>
-                    <ode>
-                        <mu>8.0</mu>
-                        <mu2>0.5</mu2>
-                    </ode>
-                </friction>
-            </surface>
-        </collision>
-        <xacro:inertial_cylinder mass="2.0" length="0.1" radius="0.15">
+        </collision>
+        <xacro:inertial_cylinder mass="1.5" length="0.1" radius="0.15">
             <origin xyz="0 0 0" rpy="0 0 0"/>
         </xacro:inertial_cylinder>
@@ -157,6 +136,7 @@
     <gazebo reference="bl_wheel">
         <material>Gazebo/Blue</material>
-        <mu1>20.0</mu1>
-        <mu2>0.1</mu2>
+        <mu1>8.0</mu1>
+        <mu2>0.1</mu2>
+        <fdir1>1 0 0</fdir1>
         <kp>10000000.0</kp>
         <kd>1.0</kd>
@@ -181,14 +161,6 @@
                 <cylinder radius="0.15" length="0.1"/>
             </geometry>
-            <surface>
-                <friction>
-                    <ode>
-                        <mu>8.0</mu>
-                        <mu2>0.5</mu2>
-                    </ode>
-                </friction>
-            </surface>
-        </collision>
-        <xacro:inertial_cylinder mass="2.0" length="0.1" radius="0.15">
+        </collision>
+        <xacro:inertial_cylinder mass="1.5" length="0.1" radius="0.15">
             <origin xyz="0 0 0" rpy="0 0 0"/>
         </xacro:inertial_cylinder>
@@ -196,6 +168,7 @@
     <gazebo reference="br_wheel">
         <material>Gazebo/Blue</material>
-        <mu1>20.0</mu1>
-        <mu2>0.1</mu2>
+        <mu1>8.0</mu1>
+        <mu2>0.1</mu2>
+        <fdir1>1 0 0</fdir1>
         <kp>10000000.0</kp>
         <kd>1.0</kd>

Commit message: Decided to place the LiDAR along the z axis of the Center of Mass. Modified the collision detection, we now divide the LiDAR rays in three zones: front, left and right.

File: xacro/skid.xacro (robot description, xacro)
@@ -178,5 +178,5 @@
         <parent link="chassis"/>
         <child link="laser_frame"/>
-        <origin xyz="0.3 0 0.32" rpy="0 0 0"/> </joint>
+        <origin xyz="0.0 0 0.32" rpy="0 0 0"/> </joint>
     <link name="laser_frame">
         <visual>
